Commit message: Add custom obstacle geometry to xarm7 urdf/srdf
Co-Authored-By: Claude Sonnet 5 <noreply@anthropic.com>

File: xarm_description/urdf/xarm7/xarm7.ros2_control.xacro (robot description, xacro)
@@ -39,5 +39,7 @@
           <param name="max">3.14</param>
         </command_interface>
-        <state_interface name="position"/>
+        <state_interface name="position">
+          <param name="initial_value">1.57</param>
+        </state_interface>
         <state_interface name="velocity"/>
         <!-- <state_interface name="effort"/> -->

File: xarm_description/urdf/xarm7/xarm7.urdf.xacro (robot description, xacro)
@@ -275,4 +275,58 @@
       <dynamics damping="2" friction="1" />
     </joint>
+    <!-- Hardcoded Gripper (.stl), attached at the TCP frame (link7) -->
+    <joint name="${prefix}link7_to_gripper" type="fixed">
+      <parent link="${prefix}link7"/>
+      <child link="${prefix}gripper_link"/>
+      <origin xyz="0 0 0" rpy="0 0 1.57"/>
+    </joint>
+    <link name="${prefix}gripper_link">
+      <visual>
+        <geometry>
+          <mesh filename="package://laundry_control/meshes/xArm7_Gripper_2Plate_Assembled_RevH_ROS2_Meters.stl"/>
+        </geometry>
+        <material name="${prefix}Silver"/>
+      </visual>
+      <collision>
+        <geometry>
+          <mesh filename="package://laundry_control/meshes/xArm7_Gripper_2Plate_Assembled_RevH_ROS2_Meters.stl"/>
+        </geometry>
+      </collision>
+    </link>
+    <!-- Hardcoded Laundry Bucket (.obj) -->
+    <joint name="${prefix}base_to_bucket_joint" type="fixed">
+      <parent link="${prefix}link_base"/>
+      <child link="${prefix}laundry_bucket_link"/>
+      <origin xyz="0.14 -0.72 0.42" rpy="1.71 3.14 -3.14"/>
+    </joint>
+    <link name="${prefix}laundry_bucket_link">
+      <visual>
+        <geometry>
+          <mesh filename="package://laundry_control/meshes/bucket.obj"/>
+        </geometry>
+      </visual>
+      <collision>
+        <geometry>
+          <mesh filename="package://laundry_control/meshes/bucket.obj"/>
+        </geometry>
+      </collision>
+    </link>
+    <joint name="${prefix}base_to_automation" type="fixed">
+      <parent link="${prefix}link_base"/>
+      <child link="${prefix}table_link"/>
+      <origin xyz="0.19 -0.43 -0.02" rpy="3.14 3.14 1.57"/>
+    </joint>
+    <link name="${prefix}table_link">
+      <visual>
+        <geometry>
+          <mesh filename="package://laundry_control/meshes/table.obj"/>
+        </geometry>
+      </visual>
+      <collision>
+        <geometry>
+          <mesh filename="package://laundry_control/meshes/table.obj"/>
+        </geometry>
+      </collision>
+    </link>
     <!-- <link name="${prefix}link_eef" />
     <joint name="${prefix}joint_eef" type="fixed">

File: xarm_description/urdf/xarm7/xarm7_robot_macro.xacro (robot description, xacro)
@@ -39,5 +39,5 @@
           joint5_lower_limit="${-pi*0.99}" joint5_upper_limit="${pi*0.99}"
           joint6_lower_limit="${-1.75}" joint6_upper_limit="${pi*0.99}"
-          joint7_lower_limit="${-pi*0.99}" joint7_upper_limit="${pi*0.99}"/>
+          joint7_lower_limit="${-2.0*pi}" joint7_upper_limit="${2.0*pi}"/>
       </xacro:if>
       <xacro:xarm7_urdf prefix="${prefix}"
@@ -48,5 +48,5 @@
         joint5_lower_limit="${-pi*0.99}" joint5_upper_limit="${pi*0.99}"
         joint6_lower_limit="${-1.75}" joint6_upper_limit="${pi*0.99}"
-        joint7_lower_limit="${-pi*0.99}" joint7_upper_limit="${pi*0.99}"
+        joint7_lower_limit="${-2.0*pi}" joint7_upper_limit="${2.0*pi}"
         model_num="${model_num}"
         inertial_params_filename="${inertial_params_filename}"

File: xarm_moveit_config/srdf/_xarm7_macro.srdf.xacro (robot description, xacro)
@@ -218,4 +218,7 @@
     <disable_collisions link1="${prefix}link6" link2="${prefix}link7" reason="Adjacent" />
     <disable_collisions link1="${prefix}link7" link2="${prefix}link_eef" reason="Adjacent" />
+    <!-- hardcoded xArm7 2-plate gripper (see xarm7.urdf.xacro) -->
+    <disable_collisions link1="${prefix}link6" link2="${prefix}gripper_link" reason="Adjacent" />
+    <disable_collisions link1="${prefix}link7" link2="${prefix}gripper_link" reason="Adjacent" />
   </xacro:macro>
 </robot>
