Commit message: Drop the bucket and table from the xarm7 URDF
They are now MoveIt world collision objects added by CDE3301_Laundrobros
(laundry_control/arm/scene.py), with their poses in
laundry_control/config.py (OBSTACLES). As URDF links they were part of
the robot: MoveIt checked contact with them as self-collision, which is
never padded, and moving the bucket meant editing this package.

The gripper link, J7's +-2pi limits and J7's initial state stay.

Co-Authored-By: Claude Opus 5.5 <noreply@anthropic.com>

File: xarm_description/urdf/xarm7/xarm7.urdf.xacro (robot description, xacro)
@@ -294,39 +294,7 @@
       </collision>
     </link>
-    <!-- Hardcoded Laundry Bucket (.obj) -->
-    <joint name="${prefix}base_to_bucket_joint" type="fixed">
-      <parent link="${prefix}link_base"/>
-      <child link="${prefix}laundry_bucket_link"/>
-      <origin xyz="0.14 -0.72 0.42" rpy="1.71 3.14 -3.14"/>
-    </joint>
-    <link name="${prefix}laundry_bucket_link">
-      <visual>
-        <geometry>
-          <mesh filename="package://laundry_control/meshes/bucket.obj"/>
-        </geometry>
-      </visual>
-      <collision>
-        <geometry>
-          <mesh filename="package://laundry_control/meshes/bucket.obj"/>
-        </geometry>
-      </collision>
-    </link>
-    <joint name="${prefix}base_to_automation" type="fixed">
-      <parent link="${prefix}link_base"/>
-      <child link="${prefix}table_link"/>
-      <origin xyz="0.19 -0.43 -0.02" rpy="3.14 3.14 1.57"/>
-    </joint>
-    <link name="${prefix}table_link">
-      <visual>
-        <geometry>
-          <mesh filename="package://laundry_control/meshes/table.obj"/>
-        </geometry>
-      </visual>
-      <collision>
-        <geometry>
-          <mesh filename="package://laundry_control/meshes/table.obj"/>
-        </geometry>
-      </collision>
-    </link>
+    <!-- The laundry bucket and table are NOT robot links: CDE3301_Laundrobros
+         adds them to MoveIt as padded world collision objects, with their
+         poses set in laundry_control/config.py (OBSTACLES). -->
     <!-- <link name="${prefix}link_eef" />
     <joint name="${prefix}joint_eef" type="fixed">
